File: thingy.brd (EAGLE design)
At the start: 24 parts, among them IC1 MCP6001T-I/OT, IC2 MAX9812LEXT+T, IC3 ESP-12, IC4 ADXL345BCCZ, J1 Interface, J2 GPIO, J3 Interrupts, Q1 Electret Mic

Commit message: Add files via upload
wat is dis how 2 pley guise?
Parts:
- added CX1, CX2: 1UF/X7R, rcl:XC10B5
- added R13: 100k, resistor:R0603
- added U1: RT9013-XXXB, v-reg-new:SOT23-5
Connections:
- new net 1UF/X7R: CX1.2
- new net N$3: CX2.1, CX2.2
- new net N$5: R13.2
- net GND: now also U1.2
Changed lines of the file:
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@@
 <?xml version="1.0" encoding="utf-8"?>
 <!DOCTYPE eagle SYSTEM "eagle.dtd">
-<eagle version="6.5.0">
+<eagle version="7.7.0">
 <drawing>
 <settings>
@@
 <pass name="Default">
 <param name="RoutingGrid" value="50mil"/>
+<param name="AutoGrid" value="1"/>
+<param name="Efforts" value="0"/>
+<param name="TopRouterVariant" value="1"/>
 <param name="tpViaShape" value="round"/>
 <param name="PrefDir.1" value="|"/>
@@
 <attribute name="PACKAGE" value="0603" x="15.8353125" y="22.38375" size="0.4064" layer="27" display="off"/>
 </element>
+<element name="U1" library="v-reg-new" package="SOT23-5" value="RT9013-XXXB" x="-4.0084375" y="4.1671875"/>
+<element name="CX1" library="rcl" package="XC10B5" value="1UF/X7R" x="6.3103125" y="-7.14375"/>
+<element name="CX2" library="rcl" package="XC10B5" value="1UF/X7R" x="6.3103125" y="-22.38375"/>
+<element name="R13" library="resistor" package="R0603" value="100k" x="-4.92125" y="-37.1078125"/>
 </elements>
 <signals>
@@
 <contactref element="R8" pad="1"/>
 <contactref element="R12" pad="1"/>
+<contactref element="U1" pad="2"/>
 <wire x1="46.4740625" y1="10.95375" x2="46.4740625" y2="13.49375" width="0" layer="19" extent="1-1"/>
 <wire x1="39.6959375" y1="6.4290625" x2="46.4740625" y2="10.95375" width="0" layer="19" extent="1-1"/>
@@
 <wire x1="8.41375" y1="12.4834375" x2="10.04875" y2="8.6096875" width="0" layer="19" extent="1-1"/>
 <wire x1="7.699375" y1="16.6724375" x2="8.41375" y2="12.4834375" width="0" layer="19" extent="1-1"/>
-<wire x1="15.0353125" y1="22.38375" x2="10.04875" y2="8.6096875" width="0" layer="19" extent="1-1"/>
-<wire x1="6.594375" y1="29.5275" x2="7.699375" y2="16.6724375" width="0" layer="19" extent="1-1"/>
-<wire x1="6.8325" y1="32.0675" x2="6.594375" y2="29.5275" width="0" layer="19" extent="1-1"/>
+<wire x1="15.0353125" y1="22.38375" x2="7.699375" y2="16.6724375" width="0" layer="19" extent="1-1"/>
+<wire x1="14.4003125" y1="32.86125" x2="15.0353125" y2="22.38375" width="0" layer="19" extent="1-1"/>
+<wire x1="6.8325" y1="32.0675" x2="14.4003125" y2="32.86125" width="0" layer="19" extent="1-1"/>
+<wire x1="6.594375" y1="29.5275" x2="6.8325" y2="32.0675" width="0" layer="19" extent="1-1"/>
 <wire x1="6.9515625" y1="35.163125" x2="6.8325" y2="32.0675" width="0" layer="19" extent="1-1"/>
-<wire x1="14.4003125" y1="32.86125" x2="6.9515625" y2="35.163125" width="0" layer="19" extent="1-1"/>
+<wire x1="-4.0084375" y1="2.8670875" x2="10.04875" y2="8.6096875" width="0" layer="19" extent="1-1"/>
 </signal>
 <signal name="+3.3V">
@@
 <wire x1="6.749375" y1="16.6724375" x2="8.649375" y2="19.2844375" width="0" layer="19" extent="1-1"/>
 </signal>
+<signal name="1UF/X7R">
+<contactref element="CX1" pad="2"/>
+</signal>
+<signal name="N$3">
+<contactref element="CX2" pad="1"/>
+<contactref element="CX2" pad="2"/>
+<wire x1="11.3903125" y1="-22.38375" x2="1.2303125" y2="-22.38375" width="0" layer="19" extent="1-1"/>
+</signal>
+<signal name="N$5">
+<contactref element="R13" pad="2"/>
+</signal>
 </signals>

Commit message: Add files via upload
This can't be right..
Parts:
- removed C5: 100nF, freetronics-luke:0603
- removed IC1: MCP6001T-I/OT, burr-brown:SOT23-5
- removed IC4: ADXL345BCCZ, SparkFun:LGA14
- removed J3: Interrupts, pinhead:1X02
- removed R10, R11: 4.7kΩ, freetronics-luke:0603
- removed R2: 62kΩ, freetronics-luke:0603
- removed R3: 27kΩ, freetronics-luke:0603
- added C6, C8: 100nF, SparkFun:0402-CAP
- added C7: 10nF, SparkFun:0402-CAP
- added C9: 2,2nF, SparkFun:0402-CAP
- added IC5: MPU-6050, seb:QFN24
- added JP1: (no value), pinhead-2:1X05
- added R14, R5: (no value), SparkFun:0402-RES
Connections:
- removed net ACC_INT1: IC4.8, J3.1
- removed net ACC_INT2: IC4.9, J3.2
- removed net N$11: IC1.3, R2.1, R3.2
- removed net N$3: CX2.1, CX2.2
- new net +3V3: C7.2, C8.1, IC5.13, IC5.8, JP1.2, R14.2, R5.2
- new net INT: IC5.12, JP1.3
- new net N$2: C6.2, IC5.10
- new net N$8: C9.1, IC5.20
- new net SCL1: IC5.23, JP1.4, R5.1
- new net SDA1: IC5.24, JP1.5, R14.1
- net +3.3V: no longer C5.1, IC1.5, IC4.1, IC4.12, IC4.6, IC4.7, R10.2, R11.2, R2.2
- net GND: now also C6.1, C7.1, C8.2, C9.2, IC5.1, IC5.11, IC5.18, IC5.9, IC5.P, JP1.1; no longer C5.2, IC1.2, IC4.2, IC4.4, IC4.5, R3.1
- net N$1: now also CX2.1, CX2.2; no longer IC1.1, IC1.4
- net SCL: no longer IC4.14, R11.1
- net SDA: no longer IC4.13, R10.1

Commit message: Add files via upload
Added the MCP6001 back in woopsie
Parts:
- removed C9: 2,2nF, SparkFun:0402-CAP
- removed IC5: MPU-6050, seb:QFN24
- removed R14: (no value), SparkFun:0402-RES
- added C5: 100nF, SparkFun:0402-CAP
- added IC1: MCP6001T-I/OT, burr-brown:SOT23-5
- added IC4: MPU-6050, seb:QFN24
- added R10: (no value), SparkFun:0402-RES
- added R2: 62kΩ, freetronics-luke:0603
- added R3: 27kΩ, freetronics-luke:0603
- C6: value 100nF -> 10nF
- C7: value 10nF -> 100nF
- C8: value 100nF -> 2,2nF
- moved U1 63.8 mm to (1.59, -59.4)
- moved C6 40.9 mm to (13.2, -16.3)
- moved C7 40.9 mm to (16.3, -16.3)
- moved C8 40.9 mm to (19.4, -16.3)
- moved R5 40.4 mm to (0.67, -23.7)
- moved JP1 40.4 mm to (11.9, -7.14)
- moved CX2 26.3 mm to (11.9, -48.1)
- moved CX1 26.3 mm to (11.9, -32.9)
- moved R13 25.6 mm to (9.72, -58.1)
Connections:
- removed net N$8: C9.1, IC5.20
- new net N$11: IC1.3, R2.1, R3.2
- new net N$3: C8.1, IC4.20
- new net N$4: CX2.1, CX2.2
- net +3.3V: now also IC1.5, R2.2
- net +3V3: now also C6.2, C7.1, IC4.13, IC4.8, R10.2; no longer C7.2, C8.1, IC5.13, IC5.8, R14.2
- net GND: now also C5.1, C7.2, IC1.2, IC4.1, IC4.11, IC4.18, IC4.9, IC4.P, R3.1; no longer C7.1, C9.2, IC5.1, IC5.11, IC5.18, IC5.9, IC5.P
- net INT: now also IC4.12; no longer IC5.12
- net N$1: now also IC1.1, IC1.4; no longer CX2.1, CX2.2
- net N$2: now also C5.2, IC4.10; no longer C6.2, IC5.10
- net SCL1: now also IC4.23; no longer IC5.23
- net SDA1: now also IC4.24, R10.1; no longer IC5.24, R14.1
